File: DIJOUS_Llums_GodasJordiPerezMax.kicad_sch (KiCad schematic)
At the start: 25 parts

Commit message: Esquem
Parts:
- removed 10u, C?: C, symbol Device:C
- removed C?: 1u, symbol Device:C
- removed C?: 10n, symbol Device:C
- removed IC?: MIC5270-5.0YM5-TR, SOT95P280X145-5N, symbol LDO 6_5volts:MIC5270-5.0YM5-TR
- removed PS?: RP-1206S, RP1206S, symbol RP-1206S:RP-1206S
- added C1: 22u, symbol Device:C
- added C2, C3, C4, C5: 10n, symbol Device:C
- added J1: DE9_Plug, symbol Connector:DE9_Plug
- added J2: Conn_01x06_Socket, symbol Connector:Conn_01x06_Socket
- added L1: 2.2u, symbol Device:L
- added R1: 100k, symbol Device:R
- added U2: TPS62173DSG, Package_SON:WSON-8-1EP_2x2mm_P0.5mm_EP0.9x1.6mm_ThermalVias, symbol Regulator_Switching:TPS62173DSG
Connections:
- net +Vcc: now also C1.1, C3.1, C5.1, L1.2, R1.1, U2.6 (VOS)
- net 3.3V_sensor: now also C4.1
- net CANH_O: now also J1.2
- net CANL_O: now also J1.7
- net GND: now also C1.2, C2.2, C3.2, C4.2, C5.2, J1.3, J1.6, J2.6 (Pin_6), U2.1 (PGND), U2.4 (AGND), U2.5 (FB)
- net DC/DC_input renamed VBAT
- net VBAT: now also C2.1, U2.2 (VIN), U2.3 (EN)
- new net: L1.1, U2.7 (SW)
- new net Blinkers: J2.3 (Pin_3)
- new net Brushless: J2.5 (Pin_5)
- new net Daytime lights: J2.4 (Pin_4)
- new net High Beam: J2.2 (Pin_2)
- new net Low Beam: J2.1 (Pin_1)
- new net PG: R1.2, U2.8 (PG)
- no-connect marks 6 -> 10
Other:
- note added: "@500mA, 5V"
- note added: "OUTPUT SELECT STAGE"
- note added: "Splitting capacitor"
- note added: "The 5 pin connector is for the button panel. The other 2 pins are for Buck input and Gnd. Before Buck, we have varios components that guarantee a safe Buck input"
- note added: "The Buck converter with its conf. ensures a safe 0.5mA and 5V output for +Vcc supply. The LDO provides the 3.3V for the light sensor. The LED proves that +Vcc is working."
- note removed: "The 5 pin connector is for the button panel. The other 2 pins are for DC/DC input and Gnd. Before DC/DC, we have varios components that guarantee a safe DC/DC input"
- moved on the sheet: 1k, D?, U?
