File: Schematics/DIJOUS_Llums_GodasJordiPerezMax_v5.kicad_sch (KiCad schematic)
At the start: 74 parts, among them J1 DE9_Plug, J2 Conn_01x06_Socket, J3 Conn_01x05, J4 Conn_01x05_Socket, J5 Conn_01x02_Socket, J6 Conn_01x02, J7 Conn_01x02, J9 Conn_01x04, Q1 ZXTN19020DFFTA, Q2 ZXTN19020DFFTA, Q3 ZXTN19020DFFTA, Q4 ZXTN19020DFFTA, Q5 ZXTN19020DFFTA, Q6 ZXTN19020DFFTA, Q7 ZXTP19020DFFTA, Q8 ZXTN19020DFFTA, Q9 ZXTP19020DFFTA, U1 MCP2551-I-SN, U2 SN74LXC2T45DCUR, U4 PIC18F2580-I/SO, U5 4N25, U6 4N25, U7 ADM7172ACPZ-5.0-R7, U8 LM2596T-ADJ, U9 ADP7112ACBZ-3.3-R7, Y1 8MHz

Commit message: Update DIJOUS_Llums_GodasJordiPerezMax_v5.kicad_sch
Parts:
- removed C5: 100n, symbol Device:C
- removed Q2, Q5, Q8: ZXTN19020DFFTA, symbol ZXTN:ZXTN19020DFFTA
- removed Q7, Q9: ZXTP19020DFFTA, symbol ZXTP19020DFF:ZXTP19020DFFTA
- removed R10, R9: 1K, symbol Device:R
- removed R11, R2, R5, R7: 10K, symbol Device:R
- removed R12: TFZVTR39B, DIO_TDZVT_ROM, symbol TFZVTR39B:TFZVTR39B
- removed R6, R8: 330, symbol Device:R
- removed U5, U6: 4N25, Package_DIP:DIP-6_W7.62mm, symbol Isolator:4N25
- added D7: BZX84Cxx, Package_TO_SOT_SMD:SOT-23, symbol Diode:BZX84Cxx
- added Q5, Q7, Q8, Q9: Si7336ADP, Package_SO:PowerPAK_SO-8_Single, symbol Transistor_FET:Si7336ADP
Connections:
- net GND: now also Q7.1 (S), Q7.2 (S), Q7.3 (S), Q8.1 (S), Q8.2 (S), Q8.3 (S); no longer C12.2, C13.2, C14.2, C15.2, C16.2, C17.2, C18.2, CR1.2, R13.2, U7.6 (GND), U8.3 (GND), U8.5 (~{ON}/OFF), U9.C2 (GND)
- net VBAT: now also Q5.5 (D), Q9.5 (D)
- net at C12.1, D6.1 (K), U8.1 (VIN): now also D7.3 (K)
- net Fin_car_01: now reaches U4.25 (RB4/KBI0/AN9)
- net Fin_car_o2: now reaches U4.26 (RB5/KBI1/PGM)
- new net GNDPWR: C12.2, C13.2, C14.2, C15.2, C16.2, C17.2, C18.2, CR1.2, D7.1 (A), R13.2, U7.6 (GND), U8.3 (GND), U8.5 (~{ON}/OFF), U9.C2 (GND)
- new net Motor_in1: Q5.4 (G), Q8.4 (G)
- new net Motor_in2: Q7.4 (G), Q9.4 (G)
- new net Motor_o1: Q5.1 (S), Q5.2 (S), Q5.3 (S), Q7.5 (D)
- new net Motor_o2: Q8.5 (D), Q9.1 (S), Q9.2 (S), Q9.3 (S)
- no-connect marks 9 -> 7
Other:
- note added: "Detector final de carrera"
- note added: "For "A" turn mode, turn on Motor_in1, turn off Motor_in2. For "B" turn mode, turn on Motor_in2, turn off Motor_in1. For turn off the motor, turn off Motor_in1 and Motor_in2"
- note added: "Maximum supply voltage for Buck converter: 45V Typical peak current for Buck: 4.5 A Maximum load current for ADM7172: 2A Input voltage range for ADM7172: 2.3-6.5 V Input voltage range for ADM7112: 2.7-20V"
- note added: "This block consists of 1 Buck converter reduce voltage to 6V. Then, for ripple rejection and minimize 1 volt, there's an LDO. The output of this LDO will go to +Vcc and to another LDO, which will supply the 3.3v sensor"
- note removed: "Poner el DB-9!!!"
- moved on the sheet: Q1, Q3, Q4, Q6, RLY1
