File: Layouts/DIJOUS_Llums_GodasJordiPerezMax.kicad_pcb (KiCad board)
At the start: 0 parts

Commit message: Update DIJOUS_Llums_GodasJordiPerezMax.kicad_pcb
Primer Placement del proyecto. He hecho placement de los inputs, el buck converter y su etapa de filtrado, el puente H, el DB-9, la etapa de comunicaciones y del intranivel. Faltan algunas footprints aún, hacer todo el ruteado y establecer reglas de diseño. Si se puede capacidades en bottom, añadir las de desacoplo en bottom.
Parts:
- added C1: 100nF, Capacitor_SMD:C_1206_3216Metric_Pad1.33x1.80mm_HandSolder, F.Cu at (65.5, 120.5)
- added C11: 2.2uF, Capacitor_SMD:C_1206_3216Metric_Pad1.33x1.80mm_HandSolder, F.Cu at (71.5, 130.6)
- added C12: 47nF, Capacitor_SMD:C_1206_3216Metric_Pad1.33x1.80mm_HandSolder, F.Cu at (99.0, 29.2)
- added C13: 1nF, Capacitor_SMD:C_1206_3216Metric_Pad1.33x1.80mm_HandSolder, F.Cu at (71.5, 137.3)
- added C14: 1nF, Capacitor_SMD:C_1206_3216Metric_Pad1.33x1.80mm_HandSolder, F.Cu at (77.5, 120.5)
- added C15: 100nF, Capacitor_SMD:C_1206_3216Metric_Pad1.33x1.80mm_HandSolder, F.Cu at (77.5, 123.9)
- added C16: 4.7uF, Capacitor_SMD:C_1206_3216Metric_Pad1.33x1.80mm_HandSolder, F.Cu at (77.5, 127.2)
- added C17: 100nF, Capacitor_SMD:C_1206_3216Metric_Pad1.33x1.80mm_HandSolder, F.Cu at (88.5, 53.5)
- added C2: 56pF, Capacitor_SMD:C_1206_3216Metric_Pad1.33x1.80mm_HandSolder, F.Cu at (65.5, 123.9)
- added C3: 100nF, Capacitor_SMD:C_1206_3216Metric_Pad1.33x1.80mm_HandSolder, F.Cu at (65.5, 127.2)
- added C4: 56pF, Capacitor_SMD:C_1206_3216Metric_Pad1.33x1.80mm_HandSolder, F.Cu at (65.5, 130.6)
- added C5: 100nF, Capacitor_SMD:C_1206_3216Metric_Pad1.33x1.80mm_HandSolder, F.Cu at (65.5, 133.9)
- added C6: 100uF, Capacitor_SMD:C_1206_3216Metric_Pad1.33x1.80mm_HandSolder, F.Cu at (43.9, 36.7)
- added C7: 100nF, Capacitor_SMD:C_1206_3216Metric_Pad1.33x1.80mm_HandSolder, F.Cu at (110.0, 34.8)
- added C8: 2.2uF, Capacitor_SMD:C_1206_3216Metric_Pad1.33x1.80mm_HandSolder, F.Cu at (71.5, 123.9)
- added C9: 4.7uF, Capacitor_SMD:C_1206_3216Metric_Pad1.33x1.80mm_HandSolder, F.Cu at (69.1, 33.9)
- added D1: 1N5817, Diode_THT:D_DO-41_SOD81_P10.16mm_Horizontal, F.Cu at (123.1, 65.1)
- added D2: 1N5817, Diode_THT:D_DO-41_SOD81_P10.16mm_Horizontal, F.Cu at (139.9, 65.5)
- added D3: LED, LED_SMD:LED_1206_3216Metric, F.Cu at (94.0, 49.0)
- added D4: LED, LED_SMD:LED_1206_3216Metric, F.Cu at (99.0, 49.0)
- added D5: 1N4148, Diode_THT:D_DO-35_SOD27_P7.62mm_Horizontal, F.Cu at (43.9, 31.8)
- added D6: BZX84Cxx, Package_TO_SOT_SMD:SOT-23, F.Cu at (38.5, 37.2)
- added D7: 1N5817, Diode_THT:D_DO-41_SOD81_P10.16mm_Horizontal, F.Cu at (140.0, 49.4)
- added D9: 1N5817, Diode_THT:D_DO-41_SOD81_P10.16mm_Horizontal, F.Cu at (123.1, 49.3)
- added J1: Conn_01x05_Socket, Connector_PinHeader_1.00mm:PinHeader_1x05_P1.00mm_Vertical, F.Cu at (15.5, 59.0)
- added J10: Screw_Terminal_01x02, Connector_PinHeader_1.00mm:PinHeader_1x02_P1.00mm_Horizontal, F.Cu at (14.5, 39.1)
- added J11: Conn_01x06, Connector_PinHeader_1.00mm:PinHeader_1x06_P1.00mm_Vertical, F.Cu at (15.2, 65.7)
- added J5: Conn_01x05, Connector_PinHeader_1.00mm:PinHeader_1x05_P1.00mm_Vertical, F.Cu at (15.1, 46.0)
- added J6: Conn_01x03, Connector_PinHeader_1.00mm:PinHeader_1x03_P1.00mm_Vertical, F.Cu at (14.9, 77.7)
- added J7: Conn_01x02, Connector_PinHeader_1.00mm:PinHeader_1x02_P1.00mm_Vertical, F.Cu at (146.5, 61.5)
- added J8: DE9_Plug, Connector_Dsub:DSUB-9_Female_Horizontal_P2.77x2.54mm_EdgePinOffset9.40mm, F.Cu at (130.4, 19.5)
- added J9: Conn_01x06_Socket, Connector_PinHeader_1.00mm:PinHeader_1x06_P1.00mm_Vertical, F.Cu at (144.0, 80.5)
- added L1: 47uH, Inductor_SMD:L_Neosid_Ms42, F.Cu at (63.1, 32.1)
- added Q3: Si7336ADP, Package_SO:PowerPAK_SO-8_Single, F.Cu at (113.0, 55.7)
- added Q4: Si7336ADP, Package_SO:PowerPAK_SO-8_Single, F.Cu at (113.9, 70.1)
- added Q7: Si7336ADP, Package_SO:PowerPAK_SO-8_Single, F.Cu at (131.8, 54.2)
- added Q8: Si7336ADP, Package_SO:PowerPAK_SO-8_Single, F.Cu at (131.6, 70.6)
- added R1: 4.7k, Resistor_SMD:R_1206_3216Metric, F.Cu at (49.1, 74.5)
- added R10: 2.49k, Resistor_SMD:R_1206_3216Metric, F.Cu at (59.6, 25.7)
- added R11: 6.49k, Resistor_SMD:R_1206_3216Metric, F.Cu at (65.2, 25.5)
- added R12: 60, Resistor_THT:R_Axial_DIN0204_L3.6mm_D1.6mm_P5.08mm_Horizontal, F.Cu at (94.0, 32.2)
- added R13: 60, Resistor_THT:R_Axial_DIN0204_L3.6mm_D1.6mm_P5.08mm_Horizontal, F.Cu at (88.9, 29.7)
- added R14: 220, Resistor_SMD:R_1206_3216Metric, F.Cu at (39.9, 133.7)
- added R16: 100, Resistor_SMD:R_1206_3216Metric, F.Cu at (39.9, 136.9)
- added R17: 100, Resistor_SMD:R_1206_3216Metric, F.Cu at (39.9, 140.2)
- added R18: 100, Resistor_SMD:R_1206_3216Metric, F.Cu at (39.9, 143.5)
- added R19: 100, Resistor_SMD:R_1206_3216Metric, F.Cu at (39.9, 146.8)
- added R2: 4.7k, Resistor_SMD:R_1206_3216Metric, F.Cu at (49.6, 79.5)
- added R20: 100, Resistor_SMD:R_1206_3216Metric, F.Cu at (45.5, 120.5)
- added R21: 100, Resistor_SMD:R_1206_3216Metric, F.Cu at (45.5, 123.8)
- added R22: 100, Resistor_SMD:R_1206_3216Metric, F.Cu at (45.5, 127.1)
- added R23: 100, Resistor_SMD:R_1206_3216Metric, F.Cu at (45.5, 130.4)
- added R24: 1k, Resistor_SMD:R_1206_3216Metric, F.Cu at (25.4, 57.4)
- added R25: 1k, Resistor_SMD:R_1206_3216Metric, F.Cu at (30.6, 57.3)
- added R26: 1k, Resistor_SMD:R_1206_3216Metric, F.Cu at (35.7, 57.2)
- added R27: 1k, Resistor_SMD:R_1206_3216Metric, F.Cu at (41.5, 57.4)
- added R28: 1k, Resistor_SMD:R_1206_3216Metric, F.Cu at (47.0, 57.4)
- added R29: 1k, Resistor_SMD:R_1206_3216Metric, F.Cu at (25.0, 46.4)
- added R3: 1k, Resistor_SMD:R_1206_3216Metric, F.Cu at (94.0, 55.0)
- added R30: 1k, Resistor_SMD:R_1206_3216Metric, F.Cu at (30.2, 46.4)
- added R31: 1k, Resistor_SMD:R_1206_3216Metric, F.Cu at (35.6, 46.3)
- added R32: 1k, Resistor_SMD:R_1206_3216Metric, F.Cu at (41.3, 46.1)
- added R33: 1k, Resistor_SMD:R_1206_3216Metric, F.Cu at (24.8, 66.4)
- added R34: 1k, Resistor_SMD:R_1206_3216Metric, F.Cu at (30.0, 66.4)
- added R35: 100m, Resistor_SMD:R_0402_1005Metric, F.Cu at (83.9, 139.9)
- added R38: 10k, Resistor_SMD:R_0402_1005Metric, F.Cu at (83.9, 141.9)
- added R39: 10k, Resistor_SMD:R_0402_1005Metric, F.Cu at (83.9, 143.9)
- added R4: 4.7k, Resistor_SMD:R_1206_3216Metric, F.Cu at (69.6, 78.0)
- added R40: 1k, Resistor_SMD:R_1206_3216Metric, F.Cu at (106.0, 71.7)
- added R41: 1k, Resistor_SMD:R_1206_3216Metric, F.Cu at (106.0, 58.2)
- added R42: 1k, Resistor_SMD:R_1206_3216Metric, F.Cu at (130.0, 60.7)
- added R43: 1k, Resistor_SMD:R_1206_3216Metric, F.Cu at (145.5, 70.7)
- added R5: 1k, Resistor_SMD:R_1206_3216Metric, F.Cu at (99.0, 55.0)
- added R6: 4.7k, Resistor_SMD:R_1206_3216Metric, F.Cu at (69.5, 74.0)
- added R7: 200k, Resistor_SMD:R_1206_3216Metric, F.Cu at (69.6, 70.0)
- added R8: 100, Resistor_SMD:R_1206_3216Metric, F.Cu at (34.3, 143.5)
- added R9: 47k, Resistor_SMD:R_1206_3216Metric, F.Cu at (109.9, 39.2)
- added U2: LM2596T-ADJ, Package_TO_SOT_THT:TO-220-5_P3.4x3.7mm_StaggerOdd_Lead3.8mm_Vertical, F.Cu at (47.9, 35.8)
- added U3: PIC18F2580-I/SO, Package_SO:SOIC-28W_7.5x17.9mm_P1.27mm, F.Cu at (78.5, 53.5)
- added U4: MCP2551-I-SN, Package_SO:SOIC-8_3.9x4.9mm_P1.27mm, F.Cu at (101.0, 37.2)
- added U7: PCA9306D, Package_SO:SO-8_3.9x4.9mm_P1.27mm, F.Cu at (60.1, 74.0)
Other:
- copper layers 0 -> 2
